File: digital_supply.sch (KiCad schematic (older format))
At the start: 24 parts

Commit message: added teensy library
Parts:
- removed C?: 22u, symbol C_Small
- removed C? (x4): 0.1u, symbol C_Small
- removed C?: 4.7u, symbol C_Small
- removed R?: R_Array, symbol R_Array
- removed R?: 5R, symbol R
- removed R?: 10k, symbol R
- removed R?: 23k2, symbol R
- removed U?: MAX9611, symbol MAX9611
- added C?: 22u, symbol C_Small
- added R?: 100k, symbol R
- added R?: 10k, symbol R
- added U?: ADS1015, symbol ADS1015
- added U? (x3): ACS758, symbol ACS758
- C? (x2): value C_Small -> 10u
- R?: value 6k8 -> 50k
- R?: value 120k -> 510k
Connections:
- net labels added: 5V_MAIN, 5V_MAIN_GND, Earth, SCL_DIGSPLY, SDA_DIGSPLY
- net labels removed: SCL_MAIN, SDA_MAIN
- wire segments 156 -> 154
- no-connect marks 6 -> 3
Other:
- moved on the sheet: C?, D?, L?, R?, U?
