File: odroid.sch (KiCad schematic (older format))
At the start: 0 parts

Commit message: no idea what to write.
something :-D
Parts:
- added U?: Odroid, symbol Odroid
Connections:
- new net Earth: U?.1 (GND), U?.14 (GND), U?.20 (GND), U?.25 (GND), U?.30 (GND), U?.34 (GND), U?.39 (GND), U?.6 (I2S_SCLK), U?.9 (GND)
- new net GND5V: U?.~ (GND_Jack)
- new net SCL1: U?.5 (SCL1)
- new net SCL2: U?.28 (SCL2)
- new net SDA1: U?.3 (SDA1)
- new net SDA2: U?.27 (SDA2)
- new net VCC5V: U?.~ (GND_Jack)
Changed lines of the file:
@@
 $Descr A4 11693 8268
 encoding utf-8
-Sheet 6 7
+Sheet 6 8
 Title ""
 Date ""
@@
 Comment4 ""
 $EndDescr
-Text HLabel 1175 950  0    60   Output ~ 0
-SCL
-Text HLabel 1175 1025 0    60   BiDi ~ 0
-SDA
+Text HLabel 5775 5350 2    60   Output ~ 0
+SCL1
+Text HLabel 5775 5275 2    60   BiDi ~ 0
+SDA1
+$Comp
+L Odroid U?
+U 1 1 5895069B
+P 4325 4800
+F 0 "U?" H 4350 4825 60  0000 C CNN
+F 1 "Odroid" H 4350 4900 60  0000 C CNN
+F 2 "" H 3475 3725 60  0001 C CNN
+F 3 "" H 3475 3725 60  0001 C CNN
+	1    4325 4800
+	1    0    0    -1
+$EndComp
+Text HLabel 5775 5550 2    60   Output ~ 0
+SCL2
+Text HLabel 5775 5475 2    60   BiDi ~ 0
+SDA2
+Text HLabel 2700 4225 0    60   Input ~ 0
+VCC5V
+Text HLabel 2700 4300 0    60   Output ~ 0
+GND5V
+$Comp
+L Earth #PWR?
+U 1 1 58950D4F
+P 3100 4925
+F 0 "#PWR?" H 3100 4675 50  0001 C CNN
+F 1 "Earth" H 3100 4775 50  0001 C CNN
+F 2 "" H 3100 4925 50  0000 C CNN
+F 3 "" H 3100 4925 50  0000 C CNN
+	1    3100 4925
+	1    0    0    -1
+$EndComp
+Wire Wire Line
+	5775 5275 5400 5275
+Wire Wire Line
+	5400 5350 5775 5350
+Wire Wire Line
+	5775 5475 5400 5475
+Wire Wire Line
+	5400 5550 5775 5550
+Wire Wire Line
+	2700 4225 3375 4225
+Wire Wire Line
+	2700 4300 3375 4300
+Wire Wire Line
+	3100 4925 3100 4875
+Wire Wire Line
+	3100 4875 3375 4875
+Wire Wire Line
+	3375 4950 3300 4950
+Wire Wire Line
+	3300 3600 3300 5400
+Connection ~ 3300 4875
+Wire Wire Line
+	3300 5025 3375 5025
+Connection ~ 3300 4950
+Wire Wire Line
+	3300 5100 3375 5100
+Connection ~ 3300 5025
+Wire Wire Line
+	3300 5175 3375 5175
+Connection ~ 3300 5100
+Wire Wire Line
+	3300 5250 3375 5250
+Connection ~ 3300 5175
+Wire Wire Line
+	3300 5325 3375 5325
+Connection ~ 3300 5250
+Wire Wire Line
+	3300 5400 3375 5400
+Connection ~ 3300 5325
+Wire Wire Line
+	3375 3600 3300 3600
 $EndSCHEMATC

Commit message: added teensy library
Parts:
- added R?: R, symbol R
- added U?: Teensy3.5, symbol Teensy3.5
- added U?: TCA9548A, symbol TCA9548A
Connections:
- net labels added: GND, VCC
- net labels removed: GND5V, VCC5V
- wire segments 17 -> 48
Other:
- moved on the sheet: U?
Changed lines of the file:
@@
 LIBS:valves
 LIBS:selfmade
+LIBS:teensy
 LIBS:preamp-cache
 EELAYER 25 0
 EELAYER END
-$Descr A4 11693 8268
+$Descr A3 16535 11693
 encoding utf-8
 Sheet 6 8
@@
 Comment4 ""
 $EndDescr
-Text HLabel 5775 5350 2    60   Output ~ 0
+Text HLabel 12575 3475 2    60   Output ~ 0
 SCL1
-Text HLabel 5775 5275 2    60   BiDi ~ 0
+Text HLabel 12575 3400 2    60   BiDi ~ 0
 SDA1
 $Comp
 L Odroid U?
 U 1 1 5895069B
-P 4325 4800
-F 0 "U?" H 4350 4825 60  0000 C CNN
-F 1 "Odroid" H 4350 4900 60  0000 C CNN
-F 2 "" H 3475 3725 60  0001 C CNN
-F 3 "" H 3475 3725 60  0001 C CNN
-	1    4325 4800
-	1    0    0    -1
-$EndComp
-Text HLabel 5775 5550 2    60   Output ~ 0
+P 9025 2775
+F 0 "U?" H 9050 2800 60  0000 C CNN
+F 1 "Odroid" H 9050 2875 60  0000 C CNN
+F 2 "" H 8175 1700 60  0001 C CNN
+F 3 "" H 8175 1700 60  0001 C CNN
+	1    9025 2775
+	1    0    0    -1
+$EndComp
+Text HLabel 12425 3300 2    60   Output ~ 0
 SCL2
-Text HLabel 5775 5475 2    60   BiDi ~ 0
+Text HLabel 12425 3225 2    60   BiDi ~ 0
 SDA2
-Text HLabel 2700 4225 0    60   Input ~ 0
-VCC5V
-Text HLabel 2700 4300 0    60   Output ~ 0
-GND5V
+Text HLabel 5900 2200 0    60   Input ~ 0
+VCC
+Text HLabel 5900 2275 0    60   Output ~ 0
+GND
 $Comp
 L Earth #PWR?
 U 1 1 58950D4F
-P 3100 4925
-F 0 "#PWR?" H 3100 4675 50  0001 C CNN
-F 1 "Earth" H 3100 4775 50  0001 C CNN
-F 2 "" H 3100 4925 50  0000 C CNN
-F 3 "" H 3100 4925 50  0000 C CNN
-	1    3100 4925
-	1    0    0    -1
-$EndComp
-Wire Wire Line
-	5775 5275 5400 5275
-Wire Wire Line
-	5400 5350 5775 5350
-Wire Wire Line
-	5775 5475 5400 5475
-Wire Wire Line
-	5400 5550 5775 5550
-Wire Wire Line
-	2700 4225 3375 4225
-Wire Wire Line
-	2700 4300 3375 4300
-Wire Wire Line
-	3100 4925 3100 4875
-Wire Wire Line
-	3100 4875 3375 4875
-Wire Wire Line
-	3375 4950 3300 4950
-Wire Wire Line
-	3300 3600 3300 5400
-Connection ~ 3300 4875
-Wire Wire Line
-	3300 5025 3375 5025
-Connection ~ 3300 4950
-Wire Wire Line
-	3300 5100 3375 5100
-Connection ~ 3300 5025
-Wire Wire Line
-	3300 5175 3375 5175
-Connection ~ 3300 5100
-Wire Wire Line
-	3300 5250 3375 5250
-Connection ~ 3300 5175
-Wire Wire Line
-	3300 5325 3375 5325
-Connection ~ 3300 5250
-Wire Wire Line
-	3300 5400 3375 5400
-Connection ~ 3300 5325
-Wire Wire Line
-	3375 3600 3300 3600
+P 7800 2900
+F 0 "#PWR?" H 7800 2650 50  0001 C CNN
+F 1 "Earth" H 7800 2750 50  0001 C CNN
+F 2 "" H 7800 2900 50  0000 C CNN
+F 3 "" H 7800 2900 50  0000 C CNN
+	1    7800 2900
+	1    0    0    -1
+$EndComp
+Wire Wire Line
+	10100 3250 10400 3250
+Wire Wire Line
+	10100 3325 10475 3325
+Wire Wire Line
+	5900 2200 8075 2200
+Wire Wire Line
+	5900 2275 8075 2275
+Wire Wire Line
+	7800 2900 7800 2850
+Wire Wire Line
+	7800 2850 8075 2850
+Wire Wire Line
+	8000 2925 8075 2925
+Wire Wire Line
+	8000 1575 8000 3375
+Connection ~ 8000 2850
+Wire Wire Line
+	8000 3000 8075 3000
+Connection ~ 8000 2925
+Wire Wire Line
+	8000 3075 8075 3075
+Connection ~ 8000 3000
+Wire Wire Line
+	8000 3150 8075 3150
+Connection ~ 8000 3075
+Wire Wire Line
+	8000 3225 8075 3225
+Connection ~ 8000 3150
+Wire Wire Line
+	8000 3300 8075 3300
+Connection ~ 8000 3225
+Wire Wire Line
+	8000 3375 8075 3375
+Connection ~ 8000 3300
+Wire Wire Line
+	8075 1575 8000 1575
+$Comp
+L TCA9548A U?
+U 1 1 58AE3E91
+P 11575 2750
+F 0 "U?" H 11575 2850 60  0000 C CNN
+F 1 "TCA9548A" H 11550 2775 60  0000 C CNN
+F 2 "" H 11525 2625 60  0001 C CNN
+F 3 "" H 11525 2625 60  0001 C CNN
+	1    11575 2750
+	1    0    0    -1
+$EndComp
+Wire Wire Line
+	7550 2200 7550 1150
+Wire Wire Line
+	7550 1150 10625 1150
+Wire Wire Line
+	10625 1150 10625 2175
+Wire Wire Line
+	10625 2175 10875 2175
+Connection ~ 7550 2200
+Wire Wire Line
+	10875 2250 10550 2250
+Wire Wire Line
+	10550 1225 10550 2550
+Wire Wire Line
+	10550 1225 7650 1225
+Wire Wire Line
+	7650 1225 7650 2275
+Connection ~ 7650 2275
+Wire Wire Line
+	10400 3250 10400 2675
+Wire Wire Line
+	10400 2675 10875 2675
+Wire Wire Line
+	10475 3325 10475 2750
+Wire Wire Line
+	10475 2750 10875 2750
+Wire Wire Line
+	10550 2400 10875 2400
+Connection ~ 10550 2250
+Wire Wire Line
+	10550 2475 10875 2475
+Connection ~ 10550 2400
+Wire Wire Line
+	10550 2550 10875 2550
+Connection ~ 10550 2475
+Wire Wire Line
+	12575 3400 12300 3400
+Wire Wire Line
+	12300 3475 12575 3475
+Wire Wire Line
+	12425 3225 12300 3225
+Wire Wire Line
+	12425 3300 12300 3300
+$Comp
+L Teensy3.5 U?
+U 1 1 58A84770
+P 3950 6025
+F 0 "U?" H 3950 8325 60  0000 C CNN
+F 1 "Teensy3.5" H 3950 3725 60  0000 C CNN
+F 2 "" H 3950 6025 60  0000 C CNN
+F 3 "" H 3950 6025 60  0000 C CNN
+	1    3950 6025
+	1    0    0    -1
+$EndComp
+Wire Wire Line
+	6375 7225 4950 7225
+Wire Wire Line
+	6375 2200 6375 7225
+Connection ~ 6375 2200
+Wire Wire Line
+	4950 6325 6275 6325
+Wire Wire Line
+	6275 6325 6275 2275
+Connection ~ 6275 2275
+Wire Wire Line
+	12400 3400 12400 4825
+Wire Wire Line
+	12400 4825 4950 4825
+Connection ~ 12400 3400
+Wire Wire Line
+	4950 4925 12475 4925
+Wire Wire Line
+	12475 4925 12475 3475
+Connection ~ 12475 3475
+Wire Wire Line
+	10100 2975 10250 2975
+Wire Wire Line
+	10250 2975 10250 3925
+Wire Wire Line
+	10250 3925 4950 3925
+$Comp
+L R R?
+U 1 1 58A85225
+P 6575 3700
+F 0 "R?" V 6655 3700 50  0000 C CNN
+F 1 "R" V 6575 3700 50  0000 C CNN
+F 2 "" V 6505 3700 50  0000 C CNN
+F 3 "" H 6575 3700 50  0000 C CNN
+	1    6575 3700
+	1    0    0    -1
+$EndComp
+Wire Wire Line
+	6575 3850 6575 3925
+Connection ~ 6575 3925
+Wire Wire Line
+	6575 3550 6575 3450
+Wire Wire Line
+	6575 3450 6375 3450
+Connection ~ 6375 3450
 $EndSCHEMATC

Commit message: Weiterentwicklung des Netzteiles
Parts:
- removed U?: TCA9548A, symbol TCA9548A
Connections:
- net labels added: 5V_STDBY, 5V_STDBY_GND, I2S_DIN, I2S_DOUT, I2S_LRCLK, I2S_MCLK, I2S_SCLK
- wire segments 48 -> 36
Changed lines of the file:
@@
 $Descr A3 16535 11693
 encoding utf-8
-Sheet 6 8
+Sheet 3 12
 Title ""
 Date ""
@@
 Comment4 ""
 $EndDescr
-Text HLabel 12575 3475 2    60   Output ~ 0
+Text HLabel 10850 3325 2    60   Output ~ 0
 SCL1
-Text HLabel 12575 3400 2    60   BiDi ~ 0
+Text HLabel 10850 3250 2    60   BiDi ~ 0
 SDA1
 $Comp
@@
 	1    0    0    -1
 $EndComp
-Text HLabel 12425 3300 2    60   Output ~ 0
+Text HLabel 10325 3525 2    60   Output ~ 0
 SCL2
-Text HLabel 12425 3225 2    60   BiDi ~ 0
+Text HLabel 10325 3450 2    60   BiDi ~ 0
 SDA2
 Text HLabel 5900 2200 0    60   Input ~ 0
@@
 	1    0    0    -1
 $EndComp
-Wire Wire Line
-	10100 3250 10400 3250
-Wire Wire Line
-	10100 3325 10475 3325
 Wire Wire Line
 	5900 2200 8075 2200
@@
 Wire Wire Line
 	8075 1575 8000 1575
-$Comp
-L TCA9548A U?
-U 1 1 58AE3E91
-P 11575 2750
-F 0 "U?" H 11575 2850 60  0000 C CNN
-F 1 "TCA9548A" H 11550 2775 60  0000 C CNN
-F 2 "" H 11525 2625 60  0001 C CNN
-F 3 "" H 11525 2625 60  0001 C CNN
-	1    11575 2750
-	1    0    0    -1
-$EndComp
 Wire Wire Line
-	7550 2200 7550 1150
+	10100 3250 10850 3250
 Wire Wire Line
-	7550 1150 10625 1150
+	10100 3325 10850 3325
 Wire Wire Line
-	10625 1150 10625 2175
+	10100 3450 10325 3450
 Wire Wire Line
-	10625 2175 10875 2175
-Connection ~ 7550 2200
-Wire Wire Line
-	10875 2250 10550 2250
-Wire Wire Line
-	10550 1225 10550 2550
-Wire Wire Line
-	10550 1225 7650 1225
-Wire Wire Line
-	7650 1225 7650 2275
-Connection ~ 7650 2275
-Wire Wire Line
-	10400 3250 10400 2675
-Wire Wire Line
-	10400 2675 10875 2675
-Wire Wire Line
-	10475 3325 10475 2750
-Wire Wire Line
-	10475 2750 10875 2750
-Wire Wire Line
-	10550 2400 10875 2400
-Connection ~ 10550 2250
-Wire Wire Line
-	10550 2475 10875 2475
-Connection ~ 10550 2400
-Wire Wire Line
-	10550 2550 10875 2550
-Connection ~ 10550 2475
-Wire Wire Line
-	12575 3400 12300 3400
-Wire Wire Line
-	12300 3475 12575 3475
-Wire Wire Line
-	12425 3225 12300 3225
-Wire Wire Line
-	12425 3300 12300 3300
+	10100 3525 10325 3525
 $Comp
 L Teensy3.5 U?
@@
 $EndComp
 Wire Wire Line
-	6375 7225 4950 7225
-Wire Wire Line
-	6375 2200 6375 7225
+	6375 2200 6375 3450
 Connection ~ 6375 2200
-Wire Wire Line
-	4950 6325 6275 6325
-Wire Wire Line
-	6275 6325 6275 2275
-Connection ~ 6275 2275
-Wire Wire Line
-	12400 3400 12400 4825
-Wire Wire Line
-	12400 4825 4950 4825
-Connection ~ 12400 3400
-Wire Wire Line
-	4950 4925 12475 4925
-Wire Wire Line
-	12475 4925 12475 3475
-Connection ~ 12475 3475
 Wire Wire Line
 	10100 2975 10250 2975
@@
 Wire Wire Line
 	6575 3450 6375 3450
-Connection ~ 6375 3450
+Entry Wire Line
+	10800 3425 10900 3525
+Entry Wire Line
+	10800 3500 10900 3600
+Wire Wire Line
+	10800 3425 10800 3250
+Connection ~ 10800 3250
+Wire Wire Line
+	10800 3500 10750 3500
+Wire Wire Line
+	10750 3500 10750 3325
+Connection ~ 10750 3325
+Wire Bus Line
+	10900 3525 10900 4825
+Wire Bus Line
+	10900 4825 5275 4825
+Wire Bus Line
+	5275 4825 5275 5025
+Entry Wire Line
+	5175 4825 5275 4925
+Entry Wire Line
+	5175 4925 5275 5025
+Wire Wire Line
+	5175 4925 4950 4925
+Wire Wire Line
+	4950 4825 5175 4825
+Text HLabel 7700 1650 0    60   Input ~ 0
+I2S_DIN
+Text HLabel 7700 1800 0    60   Input ~ 0
+I2S_MCLK
+Text HLabel 7700 1875 0    60   Input ~ 0
+I2S_LRCLK
+Text HLabel 7700 1950 0    60   Input ~ 0
+I2S_SCLK
+Text HLabel 7700 2025 0    60   Input ~ 0
+I2S_DOUT
+Wire Wire Line
+	7700 1650 8075 1650
+Wire Wire Line
+	8075 1800 7700 1800
+Wire Wire Line
+	7700 1875 8075 1875
+Wire Wire Line
+	7700 1950 8075 1950
+Wire Wire Line
+	7700 2025 8075 2025
+Text HLabel 5250 7225 2    60   Input ~ 0
+5V_STDBY
+Text HLabel 5250 6425 2    60   Output ~ 0
+5V_STDBY_GND
+Wire Wire Line
+	5250 6425 4950 6425
+Wire Wire Line
+	5250 7225 4950 7225
 $EndSCHEMATC
