File: spdif_i2s.sch (KiCad schematic (older format))
At the start: 13 parts

Commit message: Odroid
Changed lines of the file:
@@
 	4200 2725 4200 2525
 Wire Wire Line
-	3475 2525 4200 2525
+	4200 2525 3475 2525
 Wire Wire Line
 	3475 2400 3475 2625
@@
 	4125 2800 4125 2600
 Wire Wire Line
-	3800 2600 4125 2600
+	4125 2600 3800 2600
 Wire Wire Line
 	3800 2400 3800 2625
