File: surge.sch (KiCad schematic (older format))
At the start: 8 parts

Commit message: no idea what to write.
something :-D
Changed lines of the file:
@@
 $Descr A4 11693 8268
 encoding utf-8
-Sheet 2 7
+Sheet 2 8
 Title ""
 Date ""
@@
 N_I
 Wire Wire Line
-	4100 3325 4300 3325
+	4100 3325 7450 3325
 Wire Wire Line
-	4300 3325 5250 3325
+	3725 3400 7450 3400
 Wire Wire Line
-	5250 3325 6550 3325
-Wire Wire Line
-	6550 3325 7450 3325
-Wire Wire Line
-	3725 3400 4475 3400
-Wire Wire Line
-	4475 3400 5625 3400
-Wire Wire Line
-	5625 3400 6750 3400
-Wire Wire Line
-	6750 3400 7450 3400
-Wire Wire Line
-	4100 3475 4650 3475
-Wire Wire Line
-	4650 3475 5875 3475
-Wire Wire Line
-	5875 3475 7000 3475
-Wire Wire Line
-	7000 3475 7450 3475
+	4100 3475 7450 3475
 Text HLabel 7450 3325 2    60   Output ~ 0
 L_O
@@
 	5625 3400 5625 4275
 Wire Wire Line
-	5250 4275 5625 4275
-Wire Wire Line
-	5625 4275 5875 4275
+	5250 4275 5875 4275
 Connection ~ 5625 3400
 $Comp
@@
 Connection ~ 4650 3475
 Wire Wire Line
-	4300 4200 4475 4200
-Wire Wire Line
-	4475 4200 4650 4200
+	4300 4200 4650 4200
 Wire Wire Line
 	4475 4200 4475 3400
@@
 $EndComp
 Wire Wire Line
-	6550 4225 6750 4225
-Wire Wire Line
-	6750 4225 7000 4225
+	6550 4225 7000 4225
 Wire Wire Line
 	6750 4225 6750 3400
