File: supply_digital.sch (KiCad schematic (older format))
At the start: 20 parts

Commit message: Weiterentwicklung des Netzteiles
Connections:
- net 5V_STDBY_GND is gone; now on net Earth: D?.4 (K), U?.1 (A0), U?.11 (GND), U?.13 (A0), U?.2 (A1), U?.2 (GND), U?.2 (GND), U?.2 (GND), U?.3 (A2), U?.4 (-Vout), U?.7 (A2), U?.8 (VSS)
- net 5V_STDBY: now also U?.10 (VDD)
- net Earth: now also U?.6 (ADDR), U?.9 (GND)
Other:
- note added: "MAIN_GND"
- note added: "STDBY_GND"
Changed lines of the file:
@@
 $Descr A4 11693 8268
 encoding utf-8
-Sheet 8 8
+Sheet 9 12
 Title ""
 Date ""
@@
 Text HLabel 1675 6075 0    60   Input ~ 0
 SCL_DIGSPLY
-Text HLabel 1675 6825 0    60   Input ~ 0
-5V_STDBY_GND
 Text HLabel 1675 6750 0    60   Output ~ 0
 5V_STDBY
 Text HLabel 1675 6550 0    60   Output ~ 0
 12V
-Text HLabel 1675 6475 0    60   Input ~ 0
-12V_GND
 Text HLabel 1650 7025 0    60   Output ~ 0
 5V_MAIN
-Text HLabel 1650 7100 0    60   Input ~ 0
-5V_MAIN_GND
 Wire Wire Line
 	2150 5800 3500 5800
@@
 	6250 1100 6250 2375
 Wire Wire Line
-	6900 2375 6900 1100
+	6900 1100 6900 2375
 Wire Wire Line
 	4200 5625 4550 5625
@@
 Connection ~ 5250 3700
 Wire Wire Line
-	2925 4975 2825 4975
-Wire Wire Line
-	2825 4975 2825 4675
+	2825 4975 2925 4975
+Wire Wire Line
+	2825 4075 2825 4975
 Wire Wire Line
 	1675 6275 2025 6275
@@
 Connection ~ 7350 5575
 Wire Wire Line
-	1675 6825 2625 6825
+	1775 6825 2625 6825
 Wire Wire Line
 	2625 6825 2625 6425
@@
 Connection ~ 6900 1200
 Wire Wire Line
-	1650 7100 2825 7100
+	1775 7100 2825 7100
 Wire Wire Line
 	2825 7100 2825 6625
@@
 	7050 2050 7050 2175
 Connection ~ 7050 2175
+Wire Wire Line
+	2925 4600 2875 4600
+Wire Wire Line
+	2875 4600 2875 4175
+Connection ~ 2875 4175
+Connection ~ 2825 4075
+Connection ~ 2825 4675
+Text HLabel 1675 6475 0    60   Input ~ 0
+GND
+Wire Wire Line
+	1775 6475 1775 7100
+Connection ~ 1775 6475
+Connection ~ 1775 6825
+Text Notes 1675 6875 2    60   ~ 0
+STDBY_GND
+Text Notes 1675 7150 2    60   ~ 0
+MAIN_GND
 $EndSCHEMATC

Commit message: blub
Connections:
- wire segments 157 -> 129
Other:
- moved on the sheet: C?, D?, R?, U?

Commit message: daily commit
Changed lines of the file:
@@
 	7175 1575 7475 1575
 Wire Wire Line
-	7475 3325 7475 1575
+	7475 1575 7475 3325
 Wire Wire Line
-	6400 3325 7475 3325
+	7475 3325 6400 3325
 Wire Wire Line
 	6400 3325 6400 3200
